File: hardware/v_simple/v_simple.kicad_pcb (KiCad board)
At the start: 2 copper layers, 32 x 42 mm, 6 parts, among them J2 locked, J3 HDR-3x1, J4 HDR-4x1, J6 HDR-3x1, X1 Arduino_pro_micro

Commit message: adding fab files of board
Parts:
- removed the G*** at (96.6, 79.2)
- added G***: LOGO, IoWLabsLogos:finn_2, B.Cu at (107.8, 66.0)
- added G***: LOGO, IoWLabsLogos:jake_2, B.Cu at (93.0, 66.4)
- J2: value locked -> HDR-4x1; footprint Connector_JST:JST_XH_B3B-XH-A_1x03_P2.50mm_Vertical -> Connector_JST:JST_XH_B4B-XH-A_1x04_P2.50mm_Vertical
- J6: footprint Connector_JST:JST_XH_B3B-XH-A_1x03_P2.50mm_Vertical -> Connector_JST:JST_XH_S3B-XH-A_1x03_P2.50mm_Horizontal; moved to B.Cu
- moved J6 7.48 mm to (94.0, 81.9)
- moved J3 0.84 mm to (97.5, 62.4)
- moved J2 0.80 mm to (103.8, 96.6)
- moved X1 0.20 mm to (85.5, 79.1)
Connections:
- J2 pad 1: /SIG -> /Tx
- J2 pad 2: /VCC -> /SIG_Rx
- J2 pad 3: /GND -> /VCC
- X1 pad 16: unconnected-(X1-Pad16) -> /Tx
- X1 pad 17: /SIG -> /SIG_Rx
Routing:
- net /SIG_Rx: track 0.00 -> 43.6 mm
- net /SIG: track 42.0 -> 0.00 mm
- net /Tx: track 0.00 -> 39.5 mm
- net /RGB: track 19.1 -> 13.7 mm
- net /VCC: track 102.5 -> 100.1 mm
- net /GND: vias 0 -> 4
- net (no net): vias 4 -> 0
Other:
- board text added: "5V"
- board text added: "EMQ-s V0.1.0 2/2022 WAC"
- board text added: "GND"
- board text added: "Modular Diagnostic Lab C+ UDD"
- board text added: "SCL"
- board text added: "SDA"
- board text added: "Tx"
