File: hardware/v_simple/v_simple.kicad_sch (KiCad schematic)
At the start: 7 parts, among them J1 AudioJack3_SwitchTR, J2 HDR-3x1, J3 HDR-3x1, J4 HDR-4x1, J5 HDR-2x1, J6 HDR-3x1, X1 Arduino_pro_micro

Commit message: adding fab files of board
Parts:
- removed J2: HDR-3x1, Connector_JST:JST_XH_B3B-XH-A_1x03_P2.50mm_Vertical, symbol IoWLabsConnectors:HDR-3x1
- added J2: HDR-4x1, Connector_JST:JST_XH_B4B-XH-A_1x04_P2.50mm_Vertical, symbol IoWLabsConnectors:HDR-4x1
- J6: footprint Connector_JST:JST_XH_B3B-XH-A_1x03_P2.50mm_Vertical -> Connector_JST:JST_XH_S3B-XH-A_1x03_P2.50mm_Horizontal
Connections:
- net GND: now also J2.4
- net VCC: now also J2.3
- net Tx: now reaches X1.16 (15)
- net Tx: now also J2.1
- net SIG renamed SIG_Rx
- net SIG_Rx: now also J2.2
Changed lines of the file:
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@@
+    (stroke (width 0) (type default) (color 0 0 0 0))
+  )
+  (wire (pts (xy 134.62 49.53) (xy 140.97 49.53))
     (stroke (width 0) (type default) (color 0 0 0 0))
   )
@@
     (stroke (width 0) (type default) (color 0 0 0 0))
   )
+  (wire (pts (xy 85.09 62.23) (xy 87.63 62.23))
+    (stroke (width 0) (type default) (color 0 0 0 0))
+  )
+  (wire (pts (xy 137.16 54.61) (xy 140.97 54.61))
+    (stroke (width 0) (type default) (color 0 0 0 0))
+  )
+  (wire (pts (xy 137.16 77.47) (xy 140.97 77.47))
+    (stroke (width 0) (type default) (color 0 0 0 0))
+  )
+  (wire (pts (xy 137.16 74.93) (xy 140.97 74.93))
+    (stroke (width 0) (type default) (color 0 0 0 0))
+  )
+  (wire (pts (xy 110.49 59.69) (xy 106.68 59.69))
+    (stroke (width 0) (type default) (color 0 0 0 0))
+  )
+  (wire (pts (xy 110.49 69.85) (xy 106.68 69.85))
+    (stroke (width 0) (type default) (color 0 0 0 0))
+  )
+  (wire (pts (xy 82.55 62.23) (xy 85.09 62.23))
+    (stroke (width 0) (type default) (color 0 0 0 0))
+  )
   (wire (pts (xy 137.16 52.07) (xy 140.97 52.07))
     (stroke (width 0) (type default) (color 0 0 0 0))
   )
-  (wire (pts (xy 85.09 62.23) (xy 87.63 62.23))
-    (stroke (width 0) (type default) (color 0 0 0 0))
-  )
-  (wire (pts (xy 137.16 77.47) (xy 140.97 77.47))
-    (stroke (width 0) (type default) (color 0 0 0 0))
-  )
-  (wire (pts (xy 137.16 74.93) (xy 140.97 74.93))
-    (stroke (width 0) (type default) (color 0 0 0 0))
-  )
-  (wire (pts (xy 110.49 59.69) (xy 106.68 59.69))
-    (stroke (width 0) (type default) (color 0 0 0 0))
-  )
-  (wire (pts (xy 110.49 69.85) (xy 106.68 69.85))
-    (stroke (width 0) (type default) (color 0 0 0 0))
-  )
-  (wire (pts (xy 82.55 62.23) (xy 85.09 62.23))
-    (stroke (width 0) (type default) (color 0 0 0 0))
-  )
   (wire (pts (xy 185.42 86.36) (xy 189.23 86.36))
     (stroke (width 0) (type default) (color 0 0 0 0))
@@
     (stroke (width 0) (type default) (color 0 0 0 0))
   )
+  (wire (pts (xy 110.49 77.47) (xy 106.68 77.47))
+    (stroke (width 0) (type default) (color 0 0 0 0))
+  )
   (wire (pts (xy 85.09 64.77) (xy 87.63 64.77))
     (stroke (width 0) (type default) (color 0 0 0 0))
@@
     (stroke (width 0) (type default) (color 0 0 0 0))
   )
-  (wire (pts (xy 137.16 54.61) (xy 140.97 54.61))
-    (stroke (width 0) (type default) (color 0 0 0 0))
-  )
-  (wire (pts (xy 137.16 49.53) (xy 140.97 49.53))
-    (stroke (width 0) (type default) (color 0 0 0 0))
-  )
   (wire (pts (xy 83.82 67.31) (xy 87.63 67.31))
     (stroke (width 0) (type default) (color 0 0 0 0))
   )
+  (wire (pts (xy 134.62 46.99) (xy 140.97 46.99))
+    (stroke (width 0) (type default) (color 0 0 0 0))
+  )
   (wire (pts (xy 135.89 82.55) (xy 140.97 82.55))
     (stroke (width 0) (type default) (color 0 0 0 0))
@@
     (effects (font (size 1.27 1.27)) (justify left bottom))
   )
+  (label "Tx" (at 110.49 77.47 0)
+    (effects (font (size 1.27 1.27)) (justify left bottom))
+  )
+  (label "VCC" (at 135.89 85.09 0)
+    (effects (font (size 1.27 1.27)) (justify left bottom))
+  )
+  (label "GND" (at 137.16 72.39 0)
+    (effects (font (size 1.27 1.27)) (justify left bottom))
+  )
+  (label "GND" (at 135.89 64.77 0)
+    (effects (font (size 1.27 1.27)) (justify left bottom))
+  )
+  (label "SIG_TEMP" (at 134.62 59.69 0)
+    (effects (font (size 1.27 1.27)) (justify left bottom))
+  )
+  (label "SCL" (at 83.82 69.85 0)
+    (effects (font (size 1.27 1.27)) (justify left bottom))
+  )
+  (label "VCC" (at 185.42 86.36 0)
+    (effects (font (size 1.27 1.27)) (justify left bottom))
+  )
+  (label "SDA" (at 83.82 67.31 0)
+    (effects (font (size 1.27 1.27)) (justify left bottom))
+  )
+  (label "VCC" (at 109.22 64.77 0)
+    (effects (font (size 1.27 1.27)) (justify left bottom))
+  )
+  (label "GND" (at 135.89 87.63 0)
+    (effects (font (size 1.27 1.27)) (justify left bottom))
+  )
+  (label "GND" (at 137.16 54.61 0)
+    (effects (font (size 1.27 1.27)) (justify left bottom))
+  )
+  (label "SCL" (at 137.16 77.47 0)
+    (effects (font (size 1.27 1.27)) (justify left bottom))
+  )
+  (label "VCC" (at 135.89 62.23 0)
+    (effects (font (size 1.27 1.27)) (justify left bottom))
+  )
   (label "VCC" (at 137.16 52.07 0)
-    (effects (font (size 1.27 1.27)) (justify left bottom))
-  )
-  (label "VCC" (at 135.89 85.09 0)
-    (effects (font (size 1.27 1.27)) (justify left bottom))
-  )
-  (label "GND" (at 137.16 72.39 0)
-    (effects (font (size 1.27 1.27)) (justify left bottom))
-  )
-  (label "GND" (at 135.89 64.77 0)
-    (effects (font (size 1.27 1.27)) (justify left bottom))
-  )
-  (label "SIG_TEMP" (at 134.62 59.69 0)
-    (effects (font (size 1.27 1.27)) (justify left bottom))
-  )
-  (label "SCL" (at 83.82 69.85 0)
-    (effects (font (size 1.27 1.27)) (justify left bottom))
-  )
-  (label "VCC" (at 185.42 86.36 0)
-    (effects (font (size 1.27 1.27)) (justify left bottom))
-  )
-  (label "SDA" (at 83.82 67.31 0)
-    (effects (font (size 1.27 1.27)) (justify left bottom))
-  )
-  (label "VCC" (at 109.22 64.77 0)
-    (effects (font (size 1.27 1.27)) (justify left bottom))
-  )
-  (label "GND" (at 135.89 87.63 0)
-    (effects (font (size 1.27 1.27)) (justify left bottom))
-  )
-  (label "SIG" (at 137.16 49.53 0)
-    (effects (font (size 1.27 1.27)) (justify left bottom))
-  )
-  (label "SCL" (at 137.16 77.47 0)
-    (effects (font (size 1.27 1.27)) (justify left bottom))
-  )
-  (label "VCC" (at 135.89 62.23 0)
     (effects (font (size 1.27 1.27)) (justify left bottom))
   )
@@
     (effects (font (size 1.27 1.27)) (justify right bottom))
   )
+  (label "SIG_Rx" (at 134.62 49.53 0)
+    (effects (font (size 1.27 1.27)) (justify left bottom))
+  )
   (label "SDA" (at 137.16 74.93 0)
     (effects (font (size 1.27 1.27)) (justify left bottom))
   )
+  (label "Tx" (at 134.62 46.99 0)
+    (effects (font (size 1.27 1.27)) (justify left bottom))
+  )
   (label "RGB" (at 135.89 82.55 0)
     (effects (font (size 1.27 1.27)) (justify left bottom))
   )
-  (label "SIG" (at 110.49 74.93 0)
+  (label "SIG_Rx" (at 110.49 74.93 0)
     (effects (font (size 1.27 1.27)) (justify left bottom))
   )
@@
   )
   (label "GND" (at 82.55 62.23 0)
-    (effects (font (size 1.27 1.27)) (justify left bottom))
-  )
-  (label "GND" (at 137.16 54.61 0)
     (effects (font (size 1.27 1.27)) (justify left bottom))
   )
@@
     (pin "3")
   )
+  (symbol (lib_id "IoWLabsConnectors:HDR-4x1") (at 143.51 46.99 0) (unit 1)
+    (in_bom yes) (on_board yes) (fields_autoplaced)
+    (property "Reference" "J2" (id 0) (at 149.86 49.5299 0)
+      (effects (font (size 1.27 1.27)) (justify left))
+    )
+    (property "Value" "HDR-4x1" (id 1) (at 149.86 52.0699 0)
+      (effects (font (size 1.27 1.27)) (justify left))
+    )
+    (property "Footprint" "Connector_JST:JST_XH_B4B-XH-A_1x04_P2.50mm_Vertical" (id 2) (at 147.32 44.45 0)
+      (effects (font (size 1.27 1.27)) hide)
+    )
+    (property "Datasheet" "" (id 3) (at 147.32 44.45 0)
+      (effects (font (size 1.27 1.27)) hide)
+    )
+    (property "Supplier" "LCSC" (id 4) (at 143.51 46.99 0)
+      (effects (font (size 1.27 1.27)) hide)
+    )
+    (pin "1")
+    (pin "2")
+    (pin "3")
+    (pin "4")
+  )
   (symbol (lib_id "IoWLabsConnectors:HDR-3x1") (at 143.51 85.09 0) (unit 1)
     (in_bom yes) (on_board yes) (fields_autoplaced)
@@
       (effects (font (size 1.27 1.27)) (justify left))
     )
-    (property "Footprint" "Connector_JST:JST_XH_B3B-XH-A_1x03_P2.50mm_Vertical" (id 2) (at 146.05 80.01 0)
+    (property "Footprint" "Connector_JST:JST_XH_S3B-XH-A_1x03_P2.50mm_Horizontal" (id 2) (at 146.05 80.01 0)
       (effects (font (size 1.27 1.27)) hide)
     )
@@
     (pin "3")
     (pin "4")
-  )
-  (symbol (lib_id "IoWLabsConnectors:HDR-3x1") (at 143.51 52.07 0) (unit 1)
-    (in_bom yes) (on_board yes) (fields_autoplaced)
-    (property "Reference" "J2" (id 0) (at 148.59 50.7999 0)
-      (effects (font (size 1.27 1.27)) (justify left))
-    )
-    (property "Value" "HDR-3x1" (id 1) (at 148.59 53.3399 0)
-      (effects (font (size 1.27 1.27)) (justify left))
-    )
-    (property "Footprint" "Connector_JST:JST_XH_B3B-XH-A_1x03_P2.50mm_Vertical" (id 2) (at 146.05 46.99 0)
-      (effects (font (size 1.27 1.27)) hide)
-    )
-    (property "Datasheet" "" (id 3) (at 146.05 46.99 0)
-      (effects (font (size 1.27 1.27)) hide)
-    )
-    (property "Supplier" "LCSC" (id 4) (at 146.05 58.42 0)
-      (effects (font (size 1.27 1.27)) hide)
-    )
-    (pin "1")
-    (pin "2")
-    (pin "3")
   )
   (symbol (lib_id "Connector:AudioJack3_SwitchTR") (at 139.7 106.68 0) (unit 1)
@@
       (reference "J1") (unit 1) (value "AudioJack3_SwitchTR") (footprint "Connector_Audio:Jack_3.5mm_Ledino_KB3SPRS_Horizontal")
     )
-    (path "/d8a31bbc-007b-4492-9c92-a92f2b006257"
-      (reference "J2") (unit 1) (value "HDR-3x1") (footprint "Connector_JST:JST_XH_B3B-XH-A_1x03_P2.50mm_Vertical")
+    (path "/794f42eb-ed24-48bf-a978-c3d7cdafb665"
+      (reference "J2") (unit 1) (value "HDR-4x1") (footprint "Connector_JST:JST_XH_B4B-XH-A_1x04_P2.50mm_Vertical")
     )
     (path "/6467ead6-1f8a-4de8-8f9b-39d9bb6b6318"
@@
     )
     (path "/853be22d-282c-4e52-bd9b-a8f63211528e"
-      (reference "J6") (unit 1) (value "HDR-3x1") (footprint "Connector_JST:JST_XH_B3B-XH-A_1x03_P2.50mm_Vertical")
+      (reference "J6") (unit 1) (value "HDR-3x1") (footprint "Connector_JST:JST_XH_S3B-XH-A_1x03_P2.50mm_Horizontal")
     )
     (path "/5dcf857d-f1ad-402b-886f-63523af8197b"
